File: v1.01Custom/Comms.kicad_sch (KiCad schematic)
At the start: 83 parts, among them J27 uSD_Socket, J43 USB, J46 ETHERNET, Q1 BC807, U13 MCP2542, U15 MCP2542, U16 KSZ8081RNACA, U17 74LVC2G125, U19 74LVC2G34, U3 EMIF06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

Commit message: Fix labels
Parts:
- R130: value 2.2K -> 1K; LCSC C144773 -> C144789; Part Number AC0402FR-072K2L -> AC0402FR-071KL
Changed lines of the file:
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@@
 			)
 		)
-		(property "Value" "2.2K"
+		(property "Value" "1K"
 			(at 65.5828 214.3252 90)
 			(effects
@@
 			)
 		)
-		(property "Part Number" "AC0402FR-072K2L"
+		(property "Part Number" "AC0402FR-071KL"
 			(at 67.31 214.63 0)
 			(effects
@@
 			)
 		)
-		(property "LCSC" "C144773"
+		(property "LCSC" "C144789"
 			(at 67.31 214.63 90)
 			(effects
