File: v1.01Custom/Duet3_MB_6XD.kicad_pcb (KiCad board)
At the start: 4 copper layers, 101.9 x 125 mm, 281 parts, among them J1 SWD, J16 EXPANSION, J17 ESP_DB, J19 A2543WV-5P, J2 A2543WV-2P, J22 A2543WV-2P, J27 uSD_Socket, J30 LASER/VFD, J33 A2543WV-4P, J34 A2543WV-4P, J43 USB, J46 ETHERNET, J48 SBC, J49 A2543WV-2P, J59 A2543WV-2P, J60 A2543WV-2P, J9 VIN, M1 FID, M11 MOUNTING, M12 Logo_KICAD, M15 MOUNTING, M2 FID, M3 MOUNTING, M9 MOUNTING, Q1 BC807, Q21 MMBTA06-7-F, Q22 MMBTA06-7-F, U1 SN74F125DR, U10 AOZ1284, U11 ATSAME70Q20B-AN, U13 MCP2542, U14 TS30041, U16 KSZ8081RNACA, U17 74LVC2G125, U19 74LVC2G34, U2 SN74F125DR, U20 Optoisolator, U21 SN74F125DR, U22 SN74F125DR, U23 Optoisolator, U24 SN74F125DR, U27 Optoisolator, U28 Optoisolator, U3 EMIF06, U4 AP7361C-33E-13, U5 RClamp0504FB, U7 AP22816AKEWT, U9 74HCT365, X1 ECS-120-10-33B-CKM-TR, X2 25Mhz

Commit message: Fix labels
Parts:
- R130, R17, R21: value 2.2K -> 1K
- R18, R9: value 75R -> 1K
Connections:
- J16 pad 3: 3.3V_EXT -> +3.3V
- J16 pad 43: 3.3V_EXT -> +3.3V
- J19 pad 1: 3.3V_EXT -> +3.3V
- R158 pad 2: 3.3V_EXT -> +3.3V
- R160 pad 2: 3.3V_EXT -> +3.3V
- R2 pad 2: 3.3V_EXT -> +3.3V
- R4 pad 2: 3.3V_EXT -> +3.3V
- R8 pad 2: 3.3V_EXT -> +3.3V
- U11 pad 130: SPI1_SCK_BUFF -> SPI1_SPCK
Routing:
- net +3.3V: track 309.8 -> 500.5 mm, vias 35 -> 37
- net 3.3V_EXT: track 190.2 -> 0.00 mm, vias 2 -> 0
- net SPI1_SPCK: track 27.9 -> 80.9 mm, vias 1 -> 4
- net spi1cs0: track 53.1 -> 54.5 mm
- net DRIVER_1_DIR: track 50.8 -> 49.4 mm
- net GRXDV: track 39.3 -> 40.1 mm
- net USB_PWR_EN: track 73.5 -> 74.1 mm
