File: v1.01Custom/Endstops.kicad_sch (KiCad schematic)
At the start: 38 parts, among them Q21 MMBTA06-7-F, Q22 MMBTA06-7-F, U20 Optoisolator, U23 Optoisolator, U27 Optoisolator, U28 Optoisolator

Commit message: Fix labels
Connections:
- net 3.3V_EXT is gone; now on net +3.3V: R158.2, R160.2, R2.2, R4.2, R8.2
