File: v1.01Custom/Headers.kicad_sch (KiCad schematic)
At the start: 62 parts, among them J1 SWD, J10 OUT_0, J11 OUT_1, J12 OUT_2, J13 TEMP_0, J14 TEMP_1, J15 TEMP_2, J16 EXPANSION, J17 ESP_DB, J19 A2543WV-5P, J2 A2543WV-2P, J20 IO_1, J21 IO_2, J22 A2543WV-2P, J23 CAN_1_OUT, J24 DRIVER_2, J25 DRIVER_1, J26 DRIVER_0, J28 SPI_DB, J3 OUT_6, J30 LASER/VFD, J31 IO_3, J33 A2543WV-4P, J34 A2543WV-4P, J35 DRIVER_3, J36 DRIVER_4, J37 DRIVER_5, J38 CAN_0_OUT, J39 PANELDUE_SD, J4 OUT_7, J41 TEMP_3, J42 DS_LED, J44 IO_7_ISO_OUT, J47 IO_8_ISO_OUT, J48 SBC, J49 A2543WV-2P, J5 OUT_8, J50 EXT_5V_IN, J51 IO_4, J53 IO_5, J54 IO_6, J55 IO_7, J56 IO_8, J59 A2543WV-2P, J6 OUT_3, J60 A2543WV-2P, J61 IO_7_ISO_IN, J62 IO_8_ISO_IN, J7 OUT_4, J8 OUT_5, J9 VIN

Commit message: Fix labels
Connections:
- net +3.3V: now also J16.3, J16.43, J19.1 (Pin_1), J20.1 (Pin_1), J21.1 (Pin_1), J31.1 (Pin_1), J51.1 (Pin_1), J53.1 (Pin_1), J54.1 (Pin_1), J55.1 (Pin_1), J56.1 (Pin_1)
- net 3.3V_EXT: no longer J16.3, J16.43, J19.1 (Pin_1), J20.1 (Pin_1), J21.1 (Pin_1), J31.1 (Pin_1), J51.1 (Pin_1), J53.1 (Pin_1), J54.1 (Pin_1), J55.1 (Pin_1), J56.1 (Pin_1)
Other:
- moved on the sheet: J19, J20, J21, J31, J51, J53, J54, J55, J56
