File: v1.01Custom/Power.kicad_sch (KiCad schematic)
At the start: 81 parts, among them U10 AOZ1284, U14 TS30041, U18 AP7330-W5-7, U4 AP7361C-33E-13

Commit message: Fix labels
Parts:
- R17: value 2.2K -> 1K; LCSC C144773 -> C144789; Part Number AC0402FR-072K2L -> AC0402FR-071KL
- R18: value 75R -> 1K; LCSC C227222 -> C144789; Part Number AC0402FR-0775RL -> AC0402FR-071KL
Changed lines of the file:
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@@
 			)
 		)
-		(property "Value" "2.2K"
+		(property "Value" "1K"
 			(at 137.9728 184.4802 90)
 			(effects
@@
 			)
 		)
-		(property "Part Number" "AC0402FR-072K2L"
+		(property "Part Number" "AC0402FR-071KL"
 			(at 139.7 184.785 0)
 			(effects
@@
 			)
 		)
-		(property "LCSC" "C144773"
+		(property "LCSC" "C144789"
 			(at 139.7 184.785 90)
 			(effects
@@
 			)
 		)
-		(property "Value" "75R"
+		(property "Value" "1K"
 			(at 149.4028 184.4802 90)
 			(effects
@@
 			)
 		)
-		(property "Part Number" " AC0402FR-0775RL"
+		(property "Part Number" "AC0402FR-071KL"
 			(at 151.13 184.785 0)
 			(effects
@@
 			)
 		)
-		(property "LCSC" "C227222"
+		(property "LCSC" "C144789"
 			(at 151.13 184.785 90)
 			(effects
