File: v1.01Custom/Processor.kicad_sch (KiCad schematic)
At the start: 78 parts, among them M1 FID, M11 MOUNTING, M12 Logo_KICAD, M15 MOUNTING, M2 FID, M3 MOUNTING, M9 MOUNTING, U11 ATSAME70Q20B-AN, X1 ECS-120-10-33B-CKM-TR

Commit message: Fix labels
Parts:
- R21: value 2.2K -> 1K; Part Number AC0402FR-072K2L -> AC0402FR-071KL
- R9: value 75R -> 1K; LCSC C227222 -> C144773; Part Number AC0402FR-0775RL -> AC0402FR-071KL
Connections:
- net SPI1_SCK_BUFF renamed SPI1_SPCK
Changed lines of the file:
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@@
 		)
 	)
+	(global_label "SPI1_SPCK"
+		(shape input)
+		(at 180.34 124.46 0)
+		(fields_autoplaced yes)
+		(effects
+			(font
+				(size 1.27 1.27)
+			)
+			(justify left)
+		)
+		(property "Intersheetrefs" "${INTERSHEET_REFS}"
+			(at 192.9519 124.46 0)
+			(effects
+				(font
+					(size 1.27 1.27)
+				)
+				(justify left)
+				(hide yes)
+			)
+		)
+	)
 	(global_label "THERMISTOR_2"
 		(shape input)
@@
 		)
 	)
-	(global_label "SPI1_SCK_BUFF"
-		(shape input)
-		(at 180.34 124.46 0)
-		(fields_autoplaced yes)
-		(effects
-			(font
-				(size 1.27 1.27)
-			)
-			(justify left)
-		)
-		(property "Intersheetrefs" "${INTERSHEET_REFS}"
-			(at 15.24 0 0)
-			(effects
-				(font
-					(size 1.27 1.27)
-				)
-				(hide yes)
-			)
-		)
-	)
 	(global_label "QSCK"
 		(shape input)
@@
 			)
 		)
-		(property "Value" "2.2K"
+		(property "Value" "1K"
 			(at 243.3828 300.6852 90)
 			(effects
@@
 			)
 		)
-		(property "Part Number" "AC0402FR-072K2L"
+		(property "Part Number" "AC0402FR-071KL"
 			(at 245.11 300.99 0)
 			(effects
@@
 			)
 		)
-		(property "Value" "75R"
+		(property "Value" "1K"
 			(at 266.2428 301.9552 90)
 			(effects
@@
 			)
 		)
-		(property "Part Number" " AC0402FR-0775RL"
+		(property "Part Number" "AC0402FR-071KL"
 			(at 267.97 302.26 0)
 			(effects
@@
 			)
 		)
-		(property "LCSC" "C227222"
+		(property "LCSC" "C144773"
 			(at 267.97 302.26 90)
 			(effects
