File: CAD/Stepper_Drv.kicad_sch (KiCad schematic)
At the start: 28 parts, among them U1 SN74F125DR, U14 SN74LVC4245APW, U2 SN74F125DR, U21 SN74F125DR, U22 SN74F125DR, U25 SN74LVC4245APW, U26 SN74LVC4245APW, U6 SN74F125DR

Commit message: Removed pull-up resistors on motor drivers and corresponding pin on the processor
also added some misc comments
I will ask one of my professors about the pull up resistors
Parts:
- removed R65, R72: 47K, Resistor_SMD:R_0402_1005Metric_Wbry, symbol Device:R_Small
Connections:
- net EN_DIR_GATE is gone; now on net GND: U14.22 (~{OE}), U26.22 (~{OE})
Other:
- note added: "ROBERT: this makes sense. Plus they a lot of ~{OE} pins, when we only want one, really."
- note removed: "It is stated that ~{OE} should be tied to VCCa with a pullup. But we need it to be low, I am unsure if we should tie a pin from the MCU directly to ~{OE} and then pullup or just tie directly to ground?"
