File: CAD/Stepper_Drv.kicad_sch (KiCad schematic)
At the start: 28 parts, among them U1 SN74F125DR, U14 SN74LVC4245APW, U2 SN74F125DR, U21 SN74F125DR, U22 SN74F125DR, U25 SN74LVC4245APW, U26 SN74LVC4245APW, U6 SN74F125DR

Commit message: Misc Changes
Parts:
- U14, U25, U26: value SN74LVC4245APW -> SN74LVC4245APWR; LCSC (none) -> C7859; RotOffset (none) -> 270
Changed lines of the file:
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@@
 			)
 		)
-		(property "Value" "SN74LVC4245APW"
+		(property "Value" "SN74LVC4245APWR"
 			(at 161.29 45.72 0)
 			(effects
@@
 				(font
 					(size 1.27 1.27)
+				)
+				(hide yes)
+			)
+		)
+		(property "RotOffset" "270"
+			(at 161.29 64.77 0)
+			(effects
+				(font
+					(size 1.524 1.524)
+				)
+				(hide yes)
+			)
+		)
+		(property "LCSC" "C7859"
+			(at 161.29 64.77 0)
+			(effects
+				(font
+					(size 1.524 1.524)
 				)
 				(hide yes)
@@
 			)
 		)
-		(property "Value" "SN74LVC4245APW"
+		(property "Value" "SN74LVC4245APWR"
 			(at 74.93 45.72 0)
 			(effects
@@
 				(font
 					(size 1.27 1.27)
+				)
+				(hide yes)
+			)
+		)
+		(property "RotOffset" "270"
+			(at 74.93 64.77 0)
+			(effects
+				(font
+					(size 1.524 1.524)
+				)
+				(hide yes)
+			)
+		)
+		(property "LCSC" "C7859"
+			(at 74.93 64.77 0)
+			(effects
+				(font
+					(size 1.524 1.524)
 				)
 				(hide yes)
@@
 			)
 		)
-		(property "Value" "SN74LVC4245APW"
+		(property "Value" "SN74LVC4245APWR"
 			(at 236.22 48.26 0)
 			(effects
@@
 				)
 				(hide yes)
+			)
+		)
+		(property "RotOffset" "270"
+			(at 236.22 67.31 0)
+			(effects
+				(font
+					(size 1.524 1.524)
+				)
+				(hide yes)
+			)
+		)
+		(property "LCSC" "C7859"
+			(at 236.22 67.31 0)
+			(effects
+				(font
+					(size 1.524 1.524)
+				)
+				(hide yes)

Commit message: Finalize changes for 1.56
LCSC and P/N updated for excessively out of stock parts.
Silkscreen changes so no more DRC errors
Parts:
- C30, C31, C32, C33, C34, C35: footprint Capacitor_SMD:C_0402_1005Metric -> 3DPotter:0402_1005Metric_NoSilk
- R65, R72, R73: footprint Resistor_SMD:R_0402_1005Metric -> 3DPotter:0402_1005Metric_NoSilk
Other:
- title: Duet 3 Main Board 3DP -> Duet 3 MB 3DP
Changed lines of the file:
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@@
 	(paper "A3" portrait)
 	(title_block
-		(title "Duet 3 Main Board 3DP")
-		(date "2026-02-17")
-		(rev "1.55")
+		(title "Duet 3 MB 3DP")
+		(date "2026-06-02")
+		(rev "1.56")
 		(company "3DPotter")
 		(comment 1 "(c) 3DPotter")
@@
 			)
 		)
-		(property "Footprint" "Capacitor_SMD:C_0402_1005Metric"
+		(property "Footprint" "3DPotter:0402_1005Metric_NoSilk"
 			(at 96.52 48.26 0)
 			(effects
@@
 			)
 		)
-		(property "Footprint" "Capacitor_SMD:C_0402_1005Metric"
+		(property "Footprint" "3DPotter:0402_1005Metric_NoSilk"
 			(at 143.51 48.26 0)
 			(effects
@@
 			)
 		)
-		(property "Footprint" "Resistor_SMD:R_0402_1005Metric"
+		(property "Footprint" "3DPotter:0402_1005Metric_NoSilk"
 			(at 130.81 48.26 0)
 			(effects
@@
 			)
 		)
-		(property "Footprint" "Capacitor_SMD:C_0402_1005Metric"
+		(property "Footprint" "3DPotter:0402_1005Metric_NoSilk"
 			(at 55.88 48.26 0)
 			(effects
@@
 			)
 		)
-		(property "Footprint" "Capacitor_SMD:C_0402_1005Metric"
+		(property "Footprint" "3DPotter:0402_1005Metric_NoSilk"
 			(at 189.23 48.26 0)
 			(effects
@@
 			)
 		)
-		(property "Footprint" "Resistor_SMD:R_0402_1005Metric"
+		(property "Footprint" "3DPotter:0402_1005Metric_NoSilk"
 			(at 204.47 50.8 0)
 			(effects
@@
 			)
 		)
-		(property "Footprint" "Resistor_SMD:R_0402_1005Metric"
+		(property "Footprint" "3DPotter:0402_1005Metric_NoSilk"
 			(at 43.18 48.26 0)
 			(effects
@@
 			)
 		)
-		(property "Footprint" "Capacitor_SMD:C_0402_1005Metric"
+		(property "Footprint" "3DPotter:0402_1005Metric_NoSilk"
 			(at 261.62 50.8 0)
 			(effects
@@
 			)
 		)
-		(property "Footprint" "Capacitor_SMD:C_0402_1005Metric"
+		(property "Footprint" "3DPotter:0402_1005Metric_NoSilk"
 			(at 215.9 50.8 0)
 			(effects
