File: CAD/Endstops.kicad_sch (KiCad schematic)
At the start: 38 parts, among them Q21 MMBTA06-7-F, Q22 MMBTA06-7-F, U20 Optoisolator, U23 Optoisolator, U27 Optoisolator, U28 Optoisolator

Commit message: WIP redoing board for new print
Removed version resistors.
Added pull-up on CMD.
Working on motors, not routed.
Added local library for custom parts.
Ran auto-cleanup of traces and vias (supervised).
Other:
- note removed: "BOM DONE"
- company: Duet3d -> 3DPotter
- title: Duet 3 Main Board 6XD -> Duet 3 Main Board 3DP

Commit message: Pin Changes / Misc
Changing some pins around so I have a chip select
Processor Pins:
PC28 ---> PA9 (Driver_2_Step)
PC29[AFE1_AD4] ---> PB1[AFE1_AD0] (TEMP_1)
PC28 -> spi1cs1
PC29 -> spi1cs2 (Unused as of now)
IDC Header:
CAN 0 Lines removed
13 -> SPI1_MOSI_BUFF
14 -> SP1_MISO
18 -> SPI1_SPCK_BUFF
19 -> spi1cs1
Misc:
Fixed all library links, should get a lot less errors now
Parts:
- D41, D46, D50, D51: footprint complib:SOD-523F -> Diode_SMD:D_SOD-523
- R1, R132, R137, R157, R158, R159, R160, R161, R162, R2, R22, R23, R3, R4, R7, R8, R98, R99: footprint Resistor_SMD:R_0402_1005Metric_Wbry -> Resistor_SMD:R_0402_1005Metric
- U20, U23, U27, U28: footprint Carters_Various_Bits_and_Pieces:SOP-4_3.8x10mm_P2.54mm -> 3DPotter:SOP254P1016X460-4N
Changed lines of the file:
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@@
 			)
 		)
-		(property "Footprint" "Resistor_SMD:R_0402_1005Metric_Wbry"
+		(property "Footprint" "Resistor_SMD:R_0402_1005Metric"
 			(at 34.29 35.56 0)
 			(effects
@@
 			)
 		)
-		(property "Footprint" "Resistor_SMD:R_0402_1005Metric_Wbry"
+		(property "Footprint" "Resistor_SMD:R_0402_1005Metric"
 			(at 40.64 27.94 0)
 			(effects
@@
 			)
 		)
-		(property "Footprint" "Resistor_SMD:R_0402_1005Metric_Wbry"
+		(property "Footprint" "Resistor_SMD:R_0402_1005Metric"
 			(at 64.77 35.56 0)
 			(effects
@@
 			)
 		)
-		(property "Footprint" "Resistor_SMD:R_0402_1005Metric_Wbry"
+		(property "Footprint" "Resistor_SMD:R_0402_1005Metric"
 			(at 71.12 27.94 0)
 			(effects
@@
 			)
 		)
-		(property "Footprint" "Resistor_SMD:R_0402_1005Metric_Wbry"
+		(property "Footprint" "Resistor_SMD:R_0402_1005Metric"
 			(at 102.87 35.56 0)
 			(effects
@@
 			)
 		)
-		(property "Footprint" "Resistor_SMD:R_0402_1005Metric_Wbry"
+		(property "Footprint" "Resistor_SMD:R_0402_1005Metric"
 			(at 109.22 27.94 0)
 			(effects
@@
 			)
 		)
-		(property "Footprint" "Resistor_SMD:R_0402_1005Metric_Wbry"
+		(property "Footprint" "Resistor_SMD:R_0402_1005Metric"
 			(at 34.29 53.34 0)
 			(effects
@@
 			)
 		)
-		(property "Footprint" "Resistor_SMD:R_0402_1005Metric_Wbry"
+		(property "Footprint" "Resistor_SMD:R_0402_1005Metric"
 			(at 151.13 43.18 0)
 			(effects
@@
 			)
 		)
-		(property "Footprint" "Resistor_SMD:R_0402_1005Metric_Wbry"
+		(property "Footprint" "Resistor_SMD:R_0402_1005Metric"
 			(at 151.13 66.04 0)
 			(effects
@@
 			)
 		)
-		(property "Footprint" "Resistor_SMD:R_0402_1005Metric_Wbry"
+		(property "Footprint" "Resistor_SMD:R_0402_1005Metric"
 			(at 30.48 76.2 0)
 			(effects
@@
 			)
 		)
-		(property "Footprint" "Resistor_SMD:R_0402_1005Metric_Wbry"
+		(property "Footprint" "Resistor_SMD:R_0402_1005Metric"
 			(at 35.56 71.12 0)
 			(effects
@@
 			)
 		)
-		(property "Footprint" "Carters_Various_Bits_and_Pieces:SOP-4_3.8x10mm_P2.54mm"
+		(property "Footprint" "3DPotter:SOP254P1016X460-4N"
 			(at 45.72 91.44 0)
 			(effects
@@
 			)
 		)
-		(property "Footprint" "complib:SOD-523F"
+		(property "Footprint" "Diode_SMD:D_SOD-523"
 			(at 52.5526 83.82 0)
 			(effects
@@
 			)
 		)
-		(property "Footprint" "Resistor_SMD:R_0402_1005Metric_Wbry"
+		(property "Footprint" "Resistor_SMD:R_0402_1005Metric"
 			(at 82.55 76.2 0)
 			(effects
@@
 			)
 		)
-		(property "Footprint" "Resistor_SMD:R_0402_1005Metric_Wbry"
+		(property "Footprint" "Resistor_SMD:R_0402_1005Metric"
 			(at 87.63 72.39 0)
 			(effects
@@
 			)
 		)
-		(property "Footprint" "Carters_Various_Bits_and_Pieces:SOP-4_3.8x10mm_P2.54mm"
+		(property "Footprint" "3DPotter:SOP254P1016X460-4N"
 			(at 97.79 92.71 0)
 			(effects
@@
 			)
 		)
-		(property "Footprint" "complib:SOD-523F"
+		(property "Footprint" "Diode_SMD:D_SOD-523"
 			(at 104.6226 85.09 0)
 			(effects
@@
 			)
 		)
-		(property "Footprint" "Carters_Various_Bits_and_Pieces:SOP-4_3.8x10mm_P2.54mm"
+		(property "Footprint" "3DPotter:SOP254P1016X460-4N"
 			(at 160.02 45.72 0)
 			(effects
@@
 			)
 		)
-		(property "Footprint" "complib:SOD-523F"
+		(property "Footprint" "Diode_SMD:D_SOD-523"
 			(at 184.6326 40.64 0)
 			(effects
@@
 			)
 		)
-		(property "Footprint" "Resistor_SMD:R_0402_1005Metric_Wbry"
+		(property "Footprint" "Resistor_SMD:R_0402_1005Metric"
 			(at 173.99 49.53 0)
 			(effects
@@
 			)
 		)
-		(property "Footprint" "Carters_Various_Bits_and_Pieces:SOP-4_3.8x10mm_P2.54mm"
+		(property "Footprint" "3DPotter:SOP254P1016X460-4N"
 			(at 160.02 68.58 0)
 			(effects
@@
 			)
 		)
-		(property "Footprint" "complib:SOD-523F"
+		(property "Footprint" "Diode_SMD:D_SOD-523"
 			(at 184.6326 63.5 0)
 			(effects
@@
 			)
 		)
-		(property "Footprint" "Resistor_SMD:R_0402_1005Metric_Wbry"
+		(property "Footprint" "Resistor_SMD:R_0402_1005Metric"
 			(at 173.99 72.39 0)
 			(effects
@@
 			)
 		)
-		(property "Footprint" "Resistor_SMD:R_0402_1005Metric_Wbry"
+		(property "Footprint" "Resistor_SMD:R_0402_1005Metric"
 			(at 40.64 45.72 0)
 			(effects
@@
 			)
 		)
-		(property "Footprint" "Resistor_SMD:R_0402_1005Metric_Wbry"
+		(property "Footprint" "Resistor_SMD:R_0402_1005Metric"
 			(at 64.77 53.34 0)
 			(effects
@@
 			)
 		)
-		(property "Footprint" "Resistor_SMD:R_0402_1005Metric_Wbry"
+		(property "Footprint" "Resistor_SMD:R_0402_1005Metric"
 			(at 71.12 45.72 0)
 			(effects

Commit message: V1.55 Pre Maufacturing
Final change for 1.55, changed connectors to jst due to board height issues with the stepper boards
DFM passed
Parts:
- U20, U23, U27, U28: PosOffset 1.9,0 -> (none); RotOffset 90 -> 0
Changed lines of the file:
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@@
 	(title_block
 		(title "Duet 3 Main Board 3DP")
-		(date "2023-02-22")
-		(rev "1.5")
+		(date "2026-02-17")
+		(rev "1.55")
 		(company "3DPotter")
 		(comment 1 "(c) 3DPotter")
@@
 			)
 		)
-		(property "RotOffset" "90"
+		(property "RotOffset" "0"
 			(at 45.72 83.82 0)
 			(effects
@@
 			)
 		)
-		(property "PosOffset" "1.9,0"
+		(property "PosOffset" ""
 			(at 45.72 83.82 0)
 			(effects
@@
 			)
 		)
-		(property "RotOffset" "90"
+		(property "RotOffset" "0"
 			(at 97.79 85.09 0)
 			(effects
@@
 			)
 		)
-		(property "PosOffset" "1.9,0"
+		(property "PosOffset" ""
 			(at 97.79 85.09 0)
 			(effects
@@
 			)
 		)
-		(property "RotOffset" "90"
+		(property "RotOffset" "0"
 			(at 160.02 38.1 0)
 			(effects
@@
 			)
 		)
-		(property "PosOffset" "1.9,0"
+		(property "PosOffset" ""
 			(at 160.02 38.1 0)
 			(effects
@@
 			)
 		)
-		(property "RotOffset" "90"
+		(property "RotOffset" "0"
 			(at 160.02 60.96 0)
 			(effects
@@
 			)
 		)
-		(property "PosOffset" "1.9,0"
+		(property "PosOffset" ""
 			(at 160.02 60.96 0)
 			(effects

Commit message: Finalize changes for 1.56
LCSC and P/N updated for excessively out of stock parts.
Silkscreen changes so no more DRC errors
Parts:
- R1, R132, R137, R157, R158, R159, R160, R161, R162, R2, R22, R23, R3, R4, R7, R8, R98, R99: footprint Resistor_SMD:R_0402_1005Metric -> 3DPotter:0402_1005Metric_NoSilk
Other:
- title: Duet 3 Main Board 3DP -> Duet 3 MB 3DP
Changed lines of the file:
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@@
 	(paper "A3" portrait)
 	(title_block
-		(title "Duet 3 Main Board 3DP")
-		(date "2026-02-17")
-		(rev "1.55")
+		(title "Duet 3 MB 3DP")
+		(date "2026-06-02")
+		(rev "1.56")
 		(company "3DPotter")
 		(comment 1 "(c) 3DPotter")
@@
 			)
 		)
-		(property "Footprint" "Resistor_SMD:R_0402_1005Metric"
+		(property "Footprint" "3DPotter:0402_1005Metric_NoSilk"
 			(at 34.29 35.56 0)
 			(effects
@@
 			)
 		)
-		(property "Footprint" "Resistor_SMD:R_0402_1005Metric"
+		(property "Footprint" "3DPotter:0402_1005Metric_NoSilk"
 			(at 40.64 27.94 0)
 			(effects
@@
 			)
 		)
-		(property "Footprint" "Resistor_SMD:R_0402_1005Metric"
+		(property "Footprint" "3DPotter:0402_1005Metric_NoSilk"
 			(at 64.77 35.56 0)
 			(effects
@@
 			)
 		)
-		(property "Footprint" "Resistor_SMD:R_0402_1005Metric"
+		(property "Footprint" "3DPotter:0402_1005Metric_NoSilk"
 			(at 71.12 27.94 0)
 			(effects
@@
 			)
 		)
-		(property "Footprint" "Resistor_SMD:R_0402_1005Metric"
+		(property "Footprint" "3DPotter:0402_1005Metric_NoSilk"
 			(at 102.87 35.56 0)
 			(effects
@@
 			)
 		)
-		(property "Footprint" "Resistor_SMD:R_0402_1005Metric"
+		(property "Footprint" "3DPotter:0402_1005Metric_NoSilk"
 			(at 109.22 27.94 0)
 			(effects
@@
 			)
 		)
-		(property "Footprint" "Resistor_SMD:R_0402_1005Metric"
+		(property "Footprint" "3DPotter:0402_1005Metric_NoSilk"
 			(at 34.29 53.34 0)
 			(effects
@@
 			)
 		)
-		(property "Footprint" "Resistor_SMD:R_0402_1005Metric"
+		(property "Footprint" "3DPotter:0402_1005Metric_NoSilk"
 			(at 151.13 43.18 0)
 			(effects
@@
 			)
 		)
-		(property "Footprint" "Resistor_SMD:R_0402_1005Metric"
+		(property "Footprint" "3DPotter:0402_1005Metric_NoSilk"
 			(at 151.13 66.04 0)
 			(effects
@@
 			)
 		)
-		(property "Footprint" "Resistor_SMD:R_0402_1005Metric"
+		(property "Footprint" "3DPotter:0402_1005Metric_NoSilk"
 			(at 30.48 76.2 0)
 			(effects
@@
 			)
 		)
-		(property "Footprint" "Resistor_SMD:R_0402_1005Metric"
+		(property "Footprint" "3DPotter:0402_1005Metric_NoSilk"
 			(at 35.56 71.12 0)
 			(effects
@@
 			)
 		)
-		(property "Footprint" "Resistor_SMD:R_0402_1005Metric"
+		(property "Footprint" "3DPotter:0402_1005Metric_NoSilk"
 			(at 82.55 76.2 0)
 			(effects
@@
 			)
 		)
-		(property "Footprint" "Resistor_SMD:R_0402_1005Metric"
+		(property "Footprint" "3DPotter:0402_1005Metric_NoSilk"
 			(at 87.63 72.39 0)
 			(effects
@@
 			)
 		)
-		(property "Footprint" "Resistor_SMD:R_0402_1005Metric"
+		(property "Footprint" "3DPotter:0402_1005Metric_NoSilk"
 			(at 173.99 49.53 0)
 			(effects
@@
 			)
 		)
-		(property "Footprint" "Resistor_SMD:R_0402_1005Metric"
+		(property "Footprint" "3DPotter:0402_1005Metric_NoSilk"
 			(at 173.99 72.39 0)
 			(effects
@@
 			)
 		)
-		(property "Footprint" "Resistor_SMD:R_0402_1005Metric"
+		(property "Footprint" "3DPotter:0402_1005Metric_NoSilk"
 			(at 40.64 45.72 0)
 			(effects
@@
 			)
 		)
-		(property "Footprint" "Resistor_SMD:R_0402_1005Metric"
+		(property "Footprint" "3DPotter:0402_1005Metric_NoSilk"
 			(at 64.77 53.34 0)
 			(effects
@@
 			)
 		)
-		(property "Footprint" "Resistor_SMD:R_0402_1005Metric"
+		(property "Footprint" "3DPotter:0402_1005Metric_NoSilk"
 			(at 71.12 45.72 0)
 			(effects
