File: CAD/Power.kicad_sch (KiCad schematic)
At the start: 92 parts, among them U10 AOZ1284, U18 AP7330-W5-7, U24 LM70860RRXR, U4 AP7361C-33E-13

Commit message: Misc Resistor changes
Parts:
- D54: footprint Diode_SMD:DFN1610-2L -> 3DPotter:DFN1610-2L
- R17: value 910R -> 5K; LCSC C227272 -> C477765; Part Number AC0402FR-07910RL -> RC0402FR-075KL
Changed lines of the file:
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@@
 			)
 		)
-		(property "Value" "910R"
+		(property "Value" "5K"
 			(at 139.2428 154.6352 90)
 			(effects
@@
 			)
 		)
-		(property "Part Number" "AC0402FR-07910RL"
+		(property "Part Number" "RC0402FR-075KL"
 			(at 140.97 154.94 0)
 			(effects
@@
 			)
 		)
-		(property "LCSC" "C227272"
+		(property "LCSC" "C477765"
 			(at 140.97 154.94 90)
 			(effects
@@
 			)
 		)
-		(property "Footprint" "Diode_SMD:DFN1610-2L"
+		(property "Footprint" "3DPotter:DFN1610-2L"
 			(at 232.41 148.59 90)
 			(effects

Commit message: Pin Changes / Misc
Changing some pins around so I have a chip select
Processor Pins:
PC28 ---> PA9 (Driver_2_Step)
PC29[AFE1_AD4] ---> PB1[AFE1_AD0] (TEMP_1)
PC28 -> spi1cs1
PC29 -> spi1cs2 (Unused as of now)
IDC Header:
CAN 0 Lines removed
13 -> SPI1_MOSI_BUFF
14 -> SP1_MISO
18 -> SPI1_SPCK_BUFF
19 -> spi1cs1
Misc:
Fixed all library links, should get a lot less errors now
Parts:
- R17, R18: footprint Resistor_SMD:R_0402_1005Metric_Wbry -> Resistor_SMD:R_0402_1005Metric
Changed lines of the file:
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@@
 			)
 		)
-		(property "Footprint" "Resistor_SMD:R_0402_1005Metric_Wbry"
+		(property "Footprint" "Resistor_SMD:R_0402_1005Metric"
 			(at 140.97 154.94 0)
 			(effects
@@
 			)
 		)
-		(property "Footprint" "Resistor_SMD:R_0402_1005Metric_Wbry"
+		(property "Footprint" "Resistor_SMD:R_0402_1005Metric"
 			(at 152.4 154.94 0)
 			(effects

Commit message: Finalize changes for 1.56
LCSC and P/N updated for excessively out of stock parts.
Silkscreen changes so no more DRC errors
Parts:
- C21: footprint Capacitor_SMD:C_0402_1005Metric -> 3DPotter:0402_1005Metric_NoSilk; LCSC C710838 -> C162095; Part Number GRM1555C1E301JA01D -> GRM1555C1H301JA01D
- C26: LCSC C2167715 -> C106243; Part Number C2012X7R2A104K125AA -> CC0805KKX7R0BB104
- C27: footprint Capacitor_SMD:C_0402_1005Metric -> 3DPotter:0402_1005Metric_NoSilk; LCSC C113049 -> C327054; Part Number GRM155R71A473KA01D -> GRM155R71A473KA01D; Alt: CC0402KRX7R6BB473
- C29, C5, C6: footprint Capacitor_SMD:C_0402_1005Metric -> 3DPotter:0402_1005Metric_NoSilk
- R17, R18, R48, R55, R61, R62, R64: footprint Resistor_SMD:R_0402_1005Metric -> 3DPotter:0402_1005Metric_NoSilk
Other:
- title: Duet 3 Main Board 3DP -> Duet 3 MB 3DP
Changed lines of the file:
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@@
 	(paper "A3" portrait)
 	(title_block
-		(title "Duet 3 Main Board 3DP")
-		(date "2026-02-17")
-		(rev "1.55")
+		(title "Duet 3 MB 3DP")
+		(date "2026-06-02")
+		(rev "1.56")
 		(company "3DPotter")
 		(comment 1 "(c) 3DPotter")
@@
 			)
 		)
-		(property "Footprint" "Resistor_SMD:R_0402_1005Metric"
+		(property "Footprint" "3DPotter:0402_1005Metric_NoSilk"
 			(at 140.97 154.94 0)
 			(effects
@@
 			)
 		)
-		(property "Footprint" "Resistor_SMD:R_0402_1005Metric"
+		(property "Footprint" "3DPotter:0402_1005Metric_NoSilk"
 			(at 152.4 154.94 0)
 			(effects
@@
 			)
 		)
-		(property "Footprint" "Resistor_SMD:R_0402_1005Metric"
+		(property "Footprint" "3DPotter:0402_1005Metric_NoSilk"
 			(at 171.45 39.37 0)
 			(effects
@@
 			)
 		)
-		(property "Footprint" "Resistor_SMD:R_0402_1005Metric"
+		(property "Footprint" "3DPotter:0402_1005Metric_NoSilk"
 			(at 161.29 77.47 0)
 			(effects
@@
 			)
 		)
-		(property "Footprint" "Capacitor_SMD:C_0402_1005Metric"
+		(property "Footprint" "3DPotter:0402_1005Metric_NoSilk"
 			(at 76.2 102.87 0)
 			(effects
@@
 			)
 		)
-		(property "Footprint" "Resistor_SMD:R_0402_1005Metric"
+		(property "Footprint" "3DPotter:0402_1005Metric_NoSilk"
 			(at 161.29 97.79 0)
 			(effects
@@
 			)
 		)
-		(property "Footprint" "Capacitor_SMD:C_0402_1005Metric"
+		(property "Footprint" "3DPotter:0402_1005Metric_NoSilk"
 			(at 49.53 77.47 0)
 			(effects
@@
 			)
 		)
-		(property "Footprint" "Capacitor_SMD:C_0402_1005Metric"
+		(property "Footprint" "3DPotter:0402_1005Metric_NoSilk"
 			(at 163.83 39.37 0)
 			(effects
@@
 			)
 		)
-		(property "Part Number" "GRM155R71A473KA01D"
+		(property "Part Number" "GRM155R71A473KA01D; Alt: CC0402KRX7R6BB473"
 			(at 163.83 39.37 0)
 			(effects
@@
 			)
 		)
-		(property "LCSC" "C113049"
+		(property "LCSC" "C327054"
 			(at 163.83 39.37 0)
 			(effects
@@
 			)
 		)
-		(property "Footprint" "Capacitor_SMD:C_0402_1005Metric"
+		(property "Footprint" "3DPotter:0402_1005Metric_NoSilk"
 			(at 97.79 102.87 0)
 			(effects
@@
 			)
 		)
-		(property "Footprint" "Resistor_SMD:R_0402_1005Metric"
+		(property "Footprint" "3DPotter:0402_1005Metric_NoSilk"
 			(at 76.2 87.63 0)
 			(effects
@@
 			)
 		)
-		(property "Part Number" "C2012X7R2A104K125AA"
+		(property "Part Number" "CC0805KKX7R0BB104"
 			(at 87.63 50.8 0)
 			(effects
@@
 			)
 		)
-		(property "LCSC" "C2167715"
+		(property "LCSC" "C106243"
 			(at 87.63 50.8 0)
 			(effects
@@
 			)
 		)
-		(property "Footprint" "Capacitor_SMD:C_0402_1005Metric"
+		(property "Footprint" "3DPotter:0402_1005Metric_NoSilk"
 			(at 83.82 95.25 0)
 			(effects
@@
 			)
 		)
-		(property "Part Number" "GRM1555C1E301JA01D"
+		(property "Part Number" "GRM1555C1H301JA01D"
 			(at 83.82 95.25 0)
 			(effects
@@
 			)
 		)
-		(property "LCSC" "C710838"
+		(property "LCSC" "C162095"
 			(at 83.82 95.25 0)
 			(effects
@@
 			)
 		)
-		(property "Footprint" "Resistor_SMD:R_0402_1005Metric"
+		(property "Footprint" "3DPotter:0402_1005Metric_NoSilk"
 			(at 44.45 77.47 0)
 			(effects

Commit message: Forgot to save
Same changes as last commit, I forgot to save before pushing
Parts:
- R60: footprint Resistor_SMD:R_0612_1632Metric -> 3DPotter:R_0612_1632Metric
Changed lines of the file:
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@@
 			)
 		)
-		(property "Footprint" "Resistor_SMD:R_0612_1632Metric"
+		(property "Footprint" "3DPotter:R_0612_1632Metric"
 			(at 198.12 46.99 0)
 			(effects
