File: CAD/Power.kicad_sch (KiCad schematic)
At the start: 92 parts, among them U10 AOZ1284, U18 AP7330-W5-7, U24 LM70860RRXR, U4 AP7361C-33E-13

Commit message: Update Alternatives for 5V converter
Parts:
- U24: Alternatives (none) -> Either LM70860(C41753413) or LM70880(C41525220) can be used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; LCSC (none) -> C41525220
Changed lines of the file:
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@@
+			)
+		)
+		(property "LCSC" "C41525220"
+			(at 105.41 39.37 0)
+			(effects
+				(font
+					(size 1.524 1.524)
+				)
+				(hide yes)
+			)
+		)
+		(property "Alternatives" "Either LM70860(C41753413) or LM70880(C41525220) can be used, whichever is cheaper."
+			(at 105.41 39.37 0)
+			(effects
+				(font
+					(size 1.524 1.524)
+				)
+				(hide yes)
 			)
 		)

Commit message: Add fuse
Add 5A glass fuse that will be preinstalled on board from manufacturer
Parts:
- added F8: 5A Fuse, symbol Device:Fuse
Connections:
- no-connect marks 1 -> 3
Other:
- moved on the sheet: F1, F10, F11, F12, F5

Commit message: Update LED resistors.
Parts:
- R16: value 35.7K -> 120K; LCSC C144666 -> C144626; Part Number AC0603FR-0735K7L -> AC0603JR-07120KL
- R18: value 1K -> 10K; LCSC C144789 -> C144807; Part Number AC0402FR-071KL -> AC0402FR-0710KL; Rating (none) -> 50V, 62.5mW
Changed lines of the file:
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@@
 	(title_block
 		(title "Duet 3 MB 3DP")
-		(date "2026-06-02")
-		(rev "1.56")
+		(date "2026-07-23")
+		(rev "1.57")
 		(company "3DPotter")
 		(comment 1 "(c) 3DPotter")
@@
 			)
 		)
-		(property "Value" "35.7K"
+		(property "Value" "120K"
 			(at 125.2728 154.6352 90)
 			(effects
@@
 			)
 		)
-		(property "Part Number" "AC0603FR-0735K7L"
+		(property "Part Number" "AC0603JR-07120KL"
 			(at 127 154.94 0)
 			(effects
@@
 			)
 		)
-		(property "LCSC" "C144666"
+		(property "LCSC" "C144626"
 			(at 127 154.94 90)
 			(effects
@@
 			)
 		)
-		(property "Value" "1K"
+		(property "Value" "10K"
 			(at 150.6728 154.6352 90)
 			(effects
@@
 			)
 		)
-		(property "Part Number" "AC0402FR-071KL"
+		(property "Part Number" "AC0402FR-0710KL"
 			(at 152.4 154.94 0)
 			(effects
@@
 			)
 		)
-		(property "LCSC" "C144789"
+		(property "Rating" "50V, 62.5mW"
+			(at 152.4 154.94 90)
+			(effects
+				(font
+					(size 1.524 1.524)
+				)
+				(hide yes)
+			)
+		)
+		(property "LCSC" "C144807"
 			(at 152.4 154.94 90)
 			(effects
