File: CAD/Comms.kicad_sch (KiCad schematic)
At the start: 88 parts, among them J27 uSD_Socket, J32 Conn_01x02, J43 USB, J46 ETHERNET, J9 Conn_01x02, Q1 BC807, U13 MCP2542, U15 MCP2542, U16 KSZ8081RNACA, U17 74LVC2G125, U19 74LVC2G34, U3 EMIF06, U5 RClamp0504FB, U7 AP22816AKEWT, X2 25Mhz

Commit message: Replace EoL Components
D5, D7, D23: SML-310TT86 is EoL, changed to TLMS1000-GS15. May be slightly brighter.
C28:GRM32ER61C476KE15L is EoL, changed to GRT32EC81C476KE13L
Parts:
- D23: LCSC C79636 -> C23070302; Part Number SML-310LTT86 -> TLMS1000-GS15
Changed lines of the file:
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@@
 			)
 		)
-		(property "Part Number" " SML-310LTT86"
+		(property "Part Number" "TLMS1000-GS15"
 			(at 67.31 227.33 0)
 			(effects
@@
 			)
 		)
-		(property "LCSC" "C79636"
+		(property "LCSC" "C23070302"
 			(at 67.31 227.33 0)
 			(effects
