File: CAD/Comms.kicad_sch (KiCad schematic)
At the start: 88 parts, among them J27 uSD_Socket, J32 Conn_01x02, J43 USB, J46 ETHERNET, J9 Conn_01x02, Q1 BC807, U13 MCP2542, U15 MCP2542, U16 KSZ8081RNACA, U17 74LVC2G125, U19 74LVC2G34, U3 EMIF06, U5 RClamp0504FB, U7 AP22816AKEWT, X2 25Mhz

Commit message: External SPI for OLSDDB done
Parts:
- removed R74: 1K, 3DPotter:0402_1005Metric_NoSilk, symbol Device:R_Small
Connections:
- net SPI1_CS1 renamed EXT_SPI_CS
Changed lines of the file:
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@@
 	)
 	(junction
-		(at 261.62 222.25)
-		(diameter 0)
-		(color 0 0 0 0)
-	)
-	(junction
 		(at 152.4 69.85)
 		(diameter 0)
@@
 	(wire
 		(pts
-			(xy 261.62 218.44) (xy 261.62 222.25)
-		)
-		(stroke
-			(width 0)
-			(type default)
-		)
-	)
-	(wire
-		(pts
 			(xy 59.69 331.47) (xy 59.69 322.58)
 		)
@@
 	(wire
 		(pts
+			(xy 261.62 218.44) (xy 261.62 222.25)
+		)
+		(stroke
+			(width 0)
+			(type default)
+		)
+	)
+	(wire
+		(pts
 			(xy 55.88 93.98) (xy 49.53 93.98)
 		)
@@
 	(wire
 		(pts
-			(xy 233.68 222.25) (xy 237.49 222.25)
-		)
-		(stroke
-			(width 0)
-			(type default)
-		)
-	)
-	(wire
-		(pts
 			(xy 187.96 124.46) (xy 187.96 116.84)
 		)
@@
 	(wire
 		(pts
+			(xy 261.62 222.25) (xy 266.7 222.25)
+		)
+		(stroke
+			(width 0)
+			(type default)
+		)
+	)
+	(wire
+		(pts
 			(xy 130.81 118.11) (xy 130.81 124.46)
 		)
@@
 	(wire
 		(pts
-			(xy 242.57 222.25) (xy 261.62 222.25)
-		)
-		(stroke
-			(width 0)
-			(type default)
-		)
-	)
-	(wire
-		(pts
 			(xy 99.06 179.07) (xy 105.41 179.07)
 		)
@@
 	(wire
 		(pts
-			(xy 261.62 222.25) (xy 269.24 222.25)
-		)
-		(stroke
-			(width 0)
-			(type default)
-		)
-	)
-	(wire
-		(pts
 			(xy 76.2 306.07) (xy 71.12 306.07)
 		)
@@
 		)
 	)
-	(global_label "spi1cs1"
-		(shape input)
-		(at 233.68 222.25 180)
-		(effects
-			(font
-				(size 1.27 1.27)
-			)
-			(justify right)
-		)
-		(property "Intersheetrefs" "${INTERSHEET_REFS}"
-			(at 233.68 222.25 0)
-			(effects
-				(font
-					(size 1.27 1.27)
-				)
-				(hide yes)
-			)
-		)
-	)
 	(global_label "5V_INT"
 		(shape input)
@@
 		)
 	)
+	(global_label "EXT_SPI_CS"
+		(shape input)
+		(at 266.7 222.25 0)
+		(fields_autoplaced yes)
+		(effects
+			(font
+				(size 1.27 1.27)
+			)
+			(justify left)
+		)
+		(property "Intersheetrefs" "${INTERSHEET_REFS}"
+			(at 279.8561 222.25 0)
+			(effects
+				(font
+					(size 1.27 1.27)
+				)
+				(justify left)
+				(hide yes)
+			)
+		)
+	)
 	(global_label "MCCDA"
 		(shape input)
@@
 		)
 	)
-	(global_label "SPI1_CS1"
-		(shape input)
-		(at 269.24 222.25 0)
-		(fields_autoplaced yes)
-		(effects
-			(font
-				(size 1.27 1.27)
-			)
-			(justify left)
-		)
-		(property "Intersheetrefs" "${INTERSHEET_REFS}"
-			(at 280.5214 222.25 0)
-			(effects
-				(font
-					(size 1.27 1.27)
-				)
-				(justify left)
-				(hide yes)
-			)
-		)
-	)
 	(global_label "CAN0_H"
 		(shape input)
@@
 					(unit 1)
 				)
-			)
-		)
-	)
-	(symbol
-		(lib_id "Device:R_Small")
-		(at 240.03 222.25 270)
-		(unit 1)
-		(exclude_from_sim no)
-		(in_bom yes)
-		(on_board yes)
-		(dnp no)
-		(property "Reference" "R74"
-			(at 245.745 221.615 90)
-			(effects
-				(font
-					(size 1.27 1.27)
-				)
-			)
-		)
-		(property "Value" "1K"
-			(at 236.22 223.52 90)
-			(effects
-				(font
-					(size 1.27 1.27)
-				)
-			)
-		)
-		(property "Footprint" "3DPotter:0402_1005Metric_NoSilk"
-			(at 240.03 222.25 0)
-			(effects
-				(font
-					(size 1.524 1.524)
-				)
-				(hide yes)
-			)
-		)
-		(property "Datasheet" ""
-			(at 240.03 222.25 0)
-			(effects
-				(font
-					(size 1.524 1.524)
-				)
-				(hide yes)
-			)
-		)
-		(property "Description" ""
-			(at 240.03 222.25 0)
-			(effects
-				(font
-					(size 1.27 1.27)
-				)
-				(hide yes)
-			)
-		)
-		(property "Part Number" "AC0402FR-071KL"
-			(at 240.03 222.25 0)
-			(effects
-				(font
-					(size 1.27 1.27)
-				)
-				(hide yes)
-			)
-		)
-		(property "LCSC" "C144789"
-			(at 240.03 222.25 90)
-			(effects
-				(font
-					(size 1.524 1.524)
-				)
-				(hide yes)
-			)
-		)
-		(pin "1"
-		)
-		(pin "2"
-		)
-		(instances
-			(project "Duet3_MB_3DP"
-				(path "/94813053-1316-4754-9fb4-4dbbf7dc780d/00000000-0000-0000-0000-00005b64a4e7"
-					(reference "R74")
-					(unit 1)
-				)
