File: CAD/Processor.kicad_sch (KiCad schematic)
At the start: 77 parts, among them M1 FID, M11 MOUNTING, M15 MOUNTING, M2 FID, M3 MOUNTING, M9 MOUNTING, U11 ATSAME70Q20B-ANT, X1 ECS-120-10-33B-CKM-TR

Commit message: Add fuse
Add 5A glass fuse that will be preinstalled on board from manufacturer
Parts:
- TM2: now left out of the parts list
Changed lines of the file:
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@@
 		(unit 1)
 		(exclude_from_sim no)
-		(in_bom yes)
+		(in_bom no)
 		(on_board yes)
 		(dnp no)

Commit message: Replace EoL Components
D5, D7, D23: SML-310TT86 is EoL, changed to TLMS1000-GS15. May be slightly brighter.
C28:GRM32ER61C476KE15L is EoL, changed to GRT32EC81C476KE13L
Parts:
- D7: LCSC C79636 -> C23070302; Part Number SML-310LTT86 -> TLMS1000-GS15
Changed lines of the file:
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@@
 			)
 		)
-		(property "Part Number" " SML-310LTT86"
+		(property "Part Number" "TLMS1000-GS15"
 			(at 245.11 312.42 0)
 			(effects
@@
 			)
 		)
-		(property "LCSC" " C79636"
+		(property "LCSC" "C23070302"
 			(at 245.11 312.42 0)
 			(effects
