File: CAD/Headers.kicad_sch (KiCad schematic)
At the start: 59 parts, among them J1 SWD, J10 OUT_0, J11 OUT_1, J12 OUT_2, J13 TEMP_0, J14 TEMP_1, J15 TEMP_2, J16 EXPANSION, J17 ESP_DB, J18 250-502/000-006, J19 A2543WV-5P, J2 A2543WV-2P, J20 IO_1, J21 IO_2, J22 A2543WV-2P, J23 CAN_1_OUT, J24 DRIVER_2, J25 DRIVER_1, J26 DRIVER_0, J28 SPI_DB, J3 OUT_6, J31 IO_3, J33 A2543WV-4P, J34 A2543WV-4P, J35 DRIVER_3, J36 DRIVER_4, J37 DRIVER_5, J38 CAN_0_OUT, J39 PANELDUE_SD, J4 OUT_7, J41 TEMP_3, J42 DS_LED, J44 IO_7_ISO_OUT, J47 IO_8_ISO_OUT, J48 SBC, J5 OUT_8, J50 EXT_5V_IN, J51 IO_4, J53 IO_5, J54 IO_6, J55 IO_7, J56 IO_8, J59 A2543WV-2P, J6 OUT_3, J60 A2543WV-2P, J61 IO_7_ISO_IN, J62 IO_8_ISO_IN, J7 OUT_4, J8 OUT_5

Commit message: External SPI for the OLSDDB WIP
Connections:
- net SPI1_MISO: no longer J16.14
- net SPI1_MOSI_BUFF: no longer J16.13
- net SPI1_SPCK_BUFF: no longer J16.18
- net SPI1_CS1 renamed EXT_SPI_CS
- new net EXT_SPI_CK: J16.18
- new net EXT_SPI_DI: J16.14
- new net EXT_SPI_DO: J16.13
Changed lines of the file:
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@@
 		)
 	)
-	(global_label "SPI1_MISO"
+	(global_label "EXT_SPI_DI"
 		(shape input)
 		(at 105.41 237.49 180)
@@
 		)
 		(property "Intersheetrefs" "${INTERSHEET_REFS}"
-			(at 93.2214 237.49 0)
+			(at 92.8586 237.49 0)
 			(effects
 				(font
@@
 		)
 	)
-	(global_label "SPI1_CS1"
+	(global_label "EXT_SPI_CS"
 		(shape input)
 		(at 105.41 256.54 180)
@@
 		)
 		(property "Intersheetrefs" "${INTERSHEET_REFS}"
-			(at 94.1286 256.54 0)
+			(at 92.2539 256.54 0)
 			(effects
 				(font
@@
 		)
 	)
-	(global_label "SPI1_MOSI_BUFF"
+	(global_label "EXT_SPI_DO"
 		(shape input)
 		(at 105.41 233.68 180)
@@
 		)
 		(property "Intersheetrefs" "${INTERSHEET_REFS}"
-			(at 87.4761 233.68 0)
+			(at 92.1329 233.68 0)
 			(effects
 				(font
@@
 		)
 	)
-	(global_label "SPI1_SPCK_BUFF"
+	(global_label "EXT_SPI_CK"
 		(shape input)
 		(at 105.41 252.73 180)
@@
 		)
 		(property "Intersheetrefs" "${INTERSHEET_REFS}"
-			(at 87.0528 252.73 0)
-			(effects
-				(font
+			(at 92.1934 252.73 0)
+			(effects
+				(font
